File: hardware/sequencer.sch (KiCad schematic (older format))
At the start: 81 parts

Commit message: incremental work on main
Parts:
- SW?: value Switch_12pos -> Voice Selector
- SW?: value Switch_6pos -> Function Selector
- SW?: value Switch_6pos -> AF Selector
- SW?: value Switch_4pos -> PS Selector
- SW?: value Switch_2pos -> IF AB Selector
- SW?: value Switch_2pos -> AB Selector
Changed lines of the file:
@@
 P 5400 3250
 F 0 "SW?" H 5395 3875 60  0000 C CNN
-F 1 "Switch_12pos" H 5315 2645 60  0000 C CNN
+F 1 "Voice Selector" H 5315 2645 60  0000 C CNN
 F 2 "" H 4975 3780 60  0001 C CNN
 F 3 "" H 4975 3780 60  0001 C CNN
@@
 P 5400 4350
 F 0 "SW?" H 5400 4700 60  0000 C CNN
-F 1 "Switch_6pos" H 5400 4000 60  0000 C CNN
+F 1 "Function Selector" H 5400 4000 60  0000 C CNN
 F 2 "" H 4975 4880 60  0001 C CNN
 F 3 "" H 4975 4880 60  0001 C CNN
@@
 P 5400 5200
 F 0 "SW?" H 5400 5550 60  0000 C CNN
-F 1 "Switch_6pos" H 5400 4850 60  0000 C CNN
+F 1 "AF Selector" H 5400 4850 60  0000 C CNN
 F 2 "" H 4975 5730 60  0001 C CNN
 F 3 "" H 4975 5730 60  0001 C CNN
@@
 P 5350 6800
 F 0 "SW?" H 5348 7034 60  0000 C CNN
-F 1 "Switch_4pos" H 5354 6576 60  0000 C CNN
+F 1 "PS Selector" H 5354 6576 60  0000 C CNN
 F 2 "" H 4925 7330 60  0001 C CNN
 F 3 "" H 4925 7330 60  0001 C CNN
@@
 P 5350 6300
 F 0 "SW?" H 5346 6438 60  0000 C CNN
-F 1 "Switch_2pos" H 5360 6174 60  0000 C CNN
+F 1 "IF AB Selector" H 5360 6174 60  0000 C CNN
 F 2 "" H 4925 6830 60  0001 C CNN
 F 3 "" H 4925 6830 60  0001 C CNN
@@
 P 5350 5850
 F 0 "SW?" H 5346 5988 60  0000 C CNN
-F 1 "Switch_2pos" H 5360 5724 60  0000 C CNN
+F 1 "AB Selector" H 5360 5724 60  0000 C CNN
 F 2 "" H 4925 6380 60  0001 C CNN
 F 3 "" H 4925 6380 60  0001 C CNN
@@
 Connection ~ 5900 6750
 Wire Wire Line
-	5650 6850 6000 6850
-Connection ~ 6000 6850
-Wire Wire Line
-	5650 6950 6100 6950
-Connection ~ 6100 6950
-Wire Wire Line
 	10450 4950 10450 5100
 Wire Wire Line
@@
 Wire Wire Line
 	850  4550 850  4600
+Wire Wire Line
+	5650 6850 5900 6850
+Connection ~ 5800 6850
+Connection ~ 5900 6850
+Wire Wire Line
+	5650 6950 6000 6950
+Connection ~ 6000 6950
 $EndSCHEMATC
